File: capacitive_touch_avr.sch (EAGLE design)
At the start: 10 parts, among them J2 JACK-2.1MM

Commit message: Adding ISP and jumber at sensor R
Parts:
- added ISP: AVRISPSMD, fab:AVRISPSMD
- added JUM0, JUMR: SOLDER_JUMPER, fab:SOLDER_JUMPER
- renumbered J2 to POWER, U$1 to ATTINY, U$3 to LED, U$4 to OUPUT
Connections:
- removed net N$4: R3.2, R4.1
- new net N$1: JUM0.2, JUMR.2, R4.1
- new net N$2: JUMR.1, R3.2
- net GND: now also ISP.GND, JUM0.1
- net MISO: now also ISP.MISO
- net MOSI: now also ISP.MOSI
- net RST: now also ISP.RST
- net SCK: now also ISP.SCK
- net VCC: now also ISP.VCC
Other:
- note removed: "ISP"
- moved on the sheet: C2, R3
